Commit message: URDF modified with 4 sticks + MaxVelocity LOW (0.1)

File: iiwa_description/urdf/iiwa7_pivoting.urdf.xacro (robot description, xacro)
@@ -38,5 +38,5 @@
       <origin xyz="0.8525 -0.1375 1.007" rpy="0 0 0"/>
       <geometry>
-	<box size="0.275 0.315 0.01"/>
+	<box size="0.275 0.315 0.015"/>
       </geometry>
 	<material name="red"/>
@@ -45,5 +45,5 @@
       <origin xyz="0.8525 -0.1375 1.007" rpy="0 0 0"/>
       <geometry>
-	<box size="0.275 0.315 0.01"/>
+	<box size="0.275 0.315 0.015"/>
       </geometry>
     </collision>
@@ -52,5 +52,5 @@
       <origin xyz="0.6625 0.5975 1.007" rpy="0 0 1.57"/>
       <geometry>
-	<box size="0.275 0.315 0.01"/>
+	<box size="0.275 0.315 0.015"/>
       </geometry>
 	<material name="red"/>
@@ -59,5 +59,5 @@
       <origin xyz="0.6625 0.5975 1.007" rpy="0 0 1.57"/>
       <geometry>
-	<box size="0.275 0.315 0.01"/>
+	<box size="0.275 0.315 0.015"/>
       </geometry>
     </collision>
@@ -66,12 +66,12 @@
       <origin xyz="0.6625 0.5975 1.164" rpy="0 0 1.57"/>
       <geometry>
-	<box size="0.275 0.315 0.01"/>
+	<box size="0.275 0.315 0.015"/>
       </geometry>
 	<material name="red"/>
     </visual>
     <collision>
-      <origin xyz="0.6625 0.5975 1.164" rpy="0 0 1.57"/>
+      <origin xyz="0.6625 0.5975 1.144" rpy="0 0 1.57"/>
       <geometry>
-	<box size="0.275 0.315 0.01"/>
+	<box size="0.315 0.315 0.025"/>
       </geometry>
     </collision>
@@ -80,5 +80,5 @@
       <origin xyz="0.3475 0.5975 1.007" rpy="0 0 1.57"/>
       <geometry>
-	<box size="0.275 0.315 0.01"/>
+	<box size="0.275 0.315 0.015"/>
       </geometry>
 	<material name="red"/>
@@ -87,8 +87,64 @@
       <origin xyz="0.3475 0.5975 1.007" rpy="0 0 1.57"/>
       <geometry>
-	<box size="0.275 0.315 0.01"/>
+	<box size="0.275 0.315 0.015"/>
       </geometry>
     </collision>
-</link>
+<!--stecchetta 1-->
+ <visual>
+      <origin xyz="0.515 0.47 1.007" rpy="0 0 1.57"/>
+      <geometry>
+	<box size="0.02 0.02 0.30"/>
+      </geometry>
+	<material name="red"/>
+    </visual>
+    <collision>
+      <origin xyz="0.515 0.47 1.007" rpy="0 0 1.57"/>
+      <geometry>
+	<box size="0.04 0.04 0.30"/>
+      </geometry>
+    </collision>
+<!--stecchetta 2-->
+ <visual>
+      <origin xyz="0.81 0.47 1.007" rpy="0 0 1.57"/>
+      <geometry>
+	<box size="0.02 0.02 0.30"/>
+      </geometry>
+	<material name="red"/>
+    </visual>
+    <collision>
+      <origin xyz="0.81 0.47 1.007" rpy="0 0 1.57"/>
+      <geometry>
+	<box size="0.04 0.04 0.30"/>
+      </geometry>
+    </collision>
+<!--stecchetta 3-->
+ <visual>
+      <origin xyz="0.81 0.725 1.007" rpy="0 0 1.57"/>
+      <geometry>
+	<box size="0.02 0.02 0.30"/>
+      </geometry>
+	<material name="red"/>
+    </visual>
+    <collision>
+      <origin xyz="0.81 0.725 1.007" rpy="0 0 1.57"/>
+      <geometry>
+	<box size="0.02 0.02 0.30"/>
+      </geometry>
+    </collision>
+<!--stecchetta 4-->
+ <visual>
+      <origin xyz="0.515 0.725 1.007" rpy="0 0 1.57"/>
+      <geometry>
+	<box size="0.02 0.02 0.30"/>
+      </geometry>
+	<material name="red"/>
+    </visual>
+    <collision>
+      <origin xyz="0.515 0.725 1.007" rpy="0 0 1.57"/>
+      <geometry>
+	<box size="0.02 0.02 0.30"/>
+      </geometry>
+    </collision>
+  </link>
   <!--iiwa-->
   <xacro:iiwa7_dummy hardware_interface="$(arg hardware_interface)" robot_name="$(arg robot_name)" parent="world">

File: iiwa_description/urdf/iiwa7_pivoting.xacro (robot description, xacro)
@@ -379,5 +379,5 @@
       <parent link="${robot_name}_link_7"/>
       <child link="${robot_name}_link_ee"/>
-      <origin rpy="0 -1.57 0" xyz="0 0 0.18"/> <!--xyz="0 0 0.21"/-->
+      <origin rpy="0 -1.57 0" xyz="0 0 0.22"/> <!--xyz="0 0 0.21"/-->
     </joint>
   <joint name="${robot_name}_joint_dummy" type="revolute">

File: iiwa_description/urdf/iiwa7_tool.urdf.xacro (robot description, xacro)
@@ -38,5 +38,5 @@
       <origin xyz="0.8525 -0.1375 1.007" rpy="0 0 0"/>
       <geometry>
-	<box size="0.275 0.315 0.01"/>
+	<box size="0.275 0.315 0.015"/>
       </geometry>
 	<material name="red"/>
@@ -45,5 +45,5 @@
       <origin xyz="0.8525 -0.1375 1.007" rpy="0 0 0"/>
       <geometry>
-	<box size="0.275 0.315 0.01"/>
+	<box size="0.275 0.315 0.015"/>
       </geometry>
     </collision>
@@ -52,5 +52,5 @@
       <origin xyz="0.6625 0.5975 1.007" rpy="0 0 1.57"/>
       <geometry>
-	<box size="0.275 0.315 0.01"/>
+	<box size="0.275 0.315 0.015"/>
       </geometry>
 	<material name="red"/>
@@ -59,5 +59,5 @@
       <origin xyz="0.6625 0.5975 1.007" rpy="0 0 1.57"/>
       <geometry>
-	<box size="0.275 0.315 0.01"/>
+	<box size="0.275 0.315 0.015"/>
       </geometry>
     </collision>
@@ -66,12 +66,12 @@
       <origin xyz="0.6625 0.5975 1.164" rpy="0 0 1.57"/>
       <geometry>
-	<box size="0.275 0.315 0.01"/>
+	<box size="0.275 0.315 0.015"/>
       </geometry>
 	<material name="red"/>
     </visual>
     <collision>
-      <origin xyz="0.6625 0.5975 1.164" rpy="0 0 1.57"/>
+      <origin xyz="0.6625 0.5975 1.144" rpy="0 0 1.57"/>
       <geometry>
-	<box size="0.275 0.315 0.01"/>
+	<box size="0.315 0.315 0.025"/>
       </geometry>
     </collision>
@@ -80,5 +80,5 @@
       <origin xyz="0.3475 0.5975 1.007" rpy="0 0 1.57"/>
       <geometry>
-	<box size="0.275 0.315 0.01"/>
+	<box size="0.275 0.315 0.015"/>
       </geometry>
 	<material name="red"/>
@@ -87,8 +87,8 @@
       <origin xyz="0.3475 0.5975 1.007" rpy="0 0 1.57"/>
       <geometry>
-	<box size="0.275 0.315 0.01"/>
+	<box size="0.275 0.315 0.015"/>
       </geometry>
     </collision>
-</link>
+  </link>
   <!--iiwa-->
   <xacro:iiwa7_dummy hardware_interface="$(arg hardware_interface)" robot_name="$(arg robot_name)" parent="world">

File: iiwa_description/urdf/iiwa7_tool.xacro (robot description, xacro)
@@ -387,5 +387,5 @@
       <parent link="${robot_name}_link_dummy"/>
       <child link="${robot_name}_link_ee"/>
-      <origin xyz="0 0 0" rpy="0 0 0"/>
+      <origin xyz="0 0 0.22" rpy="0 0 0"/>
     </joint>
   <joint name="${robot_name}_tool_joint" type="fixed">

Commit message: update xacro

File: iiwa_description/urdf/iiwa7_pivoting.urdf.xacro (robot description, xacro)
@@ -59,10 +59,10 @@
       <origin xyz="0.6625 0.5975 1.007" rpy="0 0 1.57"/>
       <geometry>
-	<box size="0.275 0.315 0.015"/>
+	<box size="0.275 0.315 0.030"/>
       </geometry>
     </collision>
 <!--mensola 3-->
  <visual>
-      <origin xyz="0.6625 0.5975 1.164" rpy="0 0 1.57"/>
+      <origin xyz="0.6625 0.5975 1.160" rpy="0 0 1.57"/>
       <geometry>
 	<box size="0.275 0.315 0.015"/>
@@ -71,5 +71,5 @@
     </visual>
     <collision>
-      <origin xyz="0.6625 0.5975 1.144" rpy="0 0 1.57"/>
+      <origin xyz="0.6625 0.5975 1.160" rpy="0 0 1.57"/>
       <geometry>
 	<box size="0.315 0.315 0.025"/>

File: iiwa_description/urdf/iiwa7_tool.urdf.xacro (robot description, xacro)
@@ -18,4 +18,5 @@
     <color rgba="0.8 0.0 0.0 1.0"/>
   </material>
+  <!-- Fix to world just for testing -->
   <!-- Fix to world just for testing -->
   <link name="world">
@@ -59,10 +60,10 @@
       <origin xyz="0.6625 0.5975 1.007" rpy="0 0 1.57"/>
       <geometry>
-	<box size="0.275 0.315 0.015"/>
+	<box size="0.275 0.315 0.030"/>
       </geometry>
     </collision>
 <!--mensola 3-->
  <visual>
-      <origin xyz="0.6625 0.5975 1.164" rpy="0 0 1.57"/>
+      <origin xyz="0.6625 0.5975 1.160" rpy="0 0 1.57"/>
       <geometry>
 	<box size="0.275 0.315 0.015"/>
@@ -71,5 +72,5 @@
     </visual>
     <collision>
-      <origin xyz="0.6625 0.5975 1.144" rpy="0 0 1.57"/>
+      <origin xyz="0.6625 0.5975 1.160" rpy="0 0 1.57"/>
       <geometry>
 	<box size="0.315 0.315 0.025"/>
@@ -90,4 +91,60 @@
       </geometry>
     </collision>
+<!--stecchetta 1-->
+ <visual>
+      <origin xyz="0.515 0.47 1.007" rpy="0 0 1.57"/>
+      <geometry>
+	<box size="0.02 0.02 0.30"/>
+      </geometry>
+	<material name="red"/>
+    </visual>
+    <collision>
+      <origin xyz="0.515 0.47 1.007" rpy="0 0 1.57"/>
+      <geometry>
+	<box size="0.04 0.04 0.30"/>
+      </geometry>
+    </collision>
+<!--stecchetta 2-->
+ <visual>
+      <origin xyz="0.81 0.47 1.007" rpy="0 0 1.57"/>
+      <geometry>
+	<box size="0.02 0.02 0.30"/>
+      </geometry>
+	<material name="red"/>
+    </visual>
+    <collision>
+      <origin xyz="0.81 0.47 1.007" rpy="0 0 1.57"/>
+      <geometry>
+	<box size="0.04 0.04 0.30"/>
+      </geometry>
+    </collision>
+<!--stecchetta 3-->
+ <visual>
+      <origin xyz="0.81 0.725 1.007" rpy="0 0 1.57"/>
+      <geometry>
+	<box size="0.02 0.02 0.30"/>
+      </geometry>
+	<material name="red"/>
+    </visual>
+    <collision>
+      <origin xyz="0.81 0.725 1.007" rpy="0 0 1.57"/>
+      <geometry>
+	<box size="0.02 0.02 0.30"/>
+      </geometry>
+    </collision>
+<!--stecchetta 4-->
+ <visual>
+      <origin xyz="0.515 0.725 1.007" rpy="0 0 1.57"/>
+      <geometry>
+	<box size="0.02 0.02 0.30"/>
+      </geometry>
+	<material name="red"/>
+    </visual>
+    <collision>
+      <origin xyz="0.515 0.725 1.007" rpy="0 0 1.57"/>
+      <geometry>
+	<box size="0.02 0.02 0.30"/>
+      </geometry>
+    </collision>
   </link>
   <!--iiwa-->
